File: hardware/ClockClock/ClockClock.kicad_pcb (KiCad board)
At the start: 2 copper layers, 1 part

Commit message: Getting board design ready for printing
Parts:
- removed REF**: Wemos-D1-mini, wemos-d1-mini:wemos-d1-mini-connectors-only
- added BUZZ1: 10k, Resistor_THT:R_Axial_DIN0204_L3.6mm_D1.6mm_P5.08mm_Horizontal, F.Cu at (111.0, 159.5)
- added J1: OLED, Connector_PinHeader_2.54mm:PinHeader_1x04_P2.54mm_Vertical, F.Cu at (103.0, 156.5)
- added J2: PWR_EN, Connector_PinHeader_2.54mm:PinHeader_1x02_P2.54mm_Vertical, F.Cu at (89.5, 156.5)
- added J3: BUZZ_CON, Connector_PinHeader_2.54mm:PinHeader_1x02_P2.54mm_Vertical, F.Cu at (84.1, 156.5)
- added J4: VIBE_CON, Connector_PinHeader_2.54mm:PinHeader_1x02_P2.54mm_Vertical, F.Cu at (78.5, 156.5)
- added J5: LED_CON, Connector_PinHeader_2.54mm:PinHeader_1x02_P2.54mm_Vertical, F.Cu at (73.0, 156.5)
- added LED1: 10k, Resistor_THT:R_Axial_DIN0204_L3.6mm_D1.6mm_P5.08mm_Horizontal, F.Cu at (111.0, 133.5)
- added Q1: irfz44l, Package_TO_SOT_THT:TO-220-3_Vertical, F.Cu at (111.0, 154.5)
- added Q2: irfz44l, Package_TO_SOT_THT:TO-220-3_Vertical, F.Cu at (111.0, 141.5)
- added Q3: irfz44l, Package_TO_SOT_THT:TO-220-3_Vertical, F.Cu at (111.0, 129.0)
- added U1: 3a_dcdc_vreg_board, 3a_dcdc_vreg_board:8_pin_header_mount, B.Cu at (85.5, 139.5)
- added U2: WeMos_mini, wemos-d1-mini:wemos-d1-mini-with-pin-header-and-connector, F.Cu at (88.3, 139.3)
- added VIBE1: 10k, Resistor_THT:R_Axial_DIN0204_L3.6mm_D1.6mm_P5.08mm_Horizontal, F.Cu at (111.0, 146.5)
Other:
- board outline added: 50.8 x 39.4 mm
- net class Default: clearance 0.2 -> 0.05; trace_width 0.25 -> 0.5; via_dia 0.8 -> 0.45; via_drill 0.4 -> 0.2
- rule pad_to_mask_clearance: 0.2 -> 0.002
- rule trace_clearance: 0.2 -> 0.05
- rule trace_min: 0.2 -> 0.006
- rule via_min_drill: 0.3 -> 0.013
- rule via_min_size: 0.4 -> 0.027
- board text added: "BUZZ"
- board text added: "LED"
- board text added: "OLED"
- board text added: "PWR_EN"
- board text added: "VIBE"
