File: hardware/ClockClock/ClockClock.sch (KiCad schematic (older format))
At the start: 8 parts

Commit message: Getting board design ready for printing
Parts:
- added J2: PWR_EN, Connector_PinHeader_2.54mm:PinHeader_1x02_P2.54mm_Vertical, symbol Connector:Conn_01x02_Male
- added J3: BUZZ_CON, Connector_PinHeader_2.54mm:PinHeader_1x02_P2.54mm_Vertical, symbol Connector:Conn_01x02_Male
- added J4: VIBE_CON, Connector_PinHeader_2.54mm:PinHeader_1x02_P2.54mm_Vertical, symbol Connector:Conn_01x02_Male
- added J5: LED_CON, Connector_PinHeader_2.54mm:PinHeader_1x02_P2.54mm_Vertical, symbol Connector:Conn_01x02_Male
- added U1: 3a_dcdc_vreg_board, 3a_dcdc_vreg_board:8_pin_header_mount, symbol myLibrary:3a_dcdc_vreg_board
- BUZZ1: renamed from BUZZ; footprint (none) -> Resistor_THT:R_Axial_DIN0204_L3.6mm_D1.6mm_P5.08mm_Horizontal
- J1: renamed from J?; footprint (none) -> Connector_PinHeader_2.54mm:PinHeader_1x04_P2.54mm_Vertical
- LED1: renamed from LED; footprint (none) -> Resistor_THT:R_Axial_DIN0204_L3.6mm_D1.6mm_P5.08mm_Horizontal
- Q1, Q2, Q3: renamed from Q?; value Q_NMOS_GDS -> irfz44l; footprint (none) -> Package_TO_SOT_THT:TO-220-3_Vertical
- U2: renamed from U?; footprint (none) -> wemos-d1-mini:wemos-d1-mini-with-pin-header-and-connector
- VIBE1: renamed from VIBE; footprint (none) -> Resistor_THT:R_Axial_DIN0204_L3.6mm_D1.6mm_P5.08mm_Horizontal
Connections:
- net labels added: +12V
- wire segments 25 -> 48
- no-connect marks 0 -> 13
