File: hardware/ClockClock.sch (KiCad schematic (older format))
At the start: 13 parts, among them J1 OLED, J2 PWR_EN, J3 BUZZ_CON, J4 VIBE_CON, J5 LED_CON, Q1 irfz44l, Q2 irfz44l, Q3 irfz44l, U1 3a_dcdc_vreg_board, U2 WeMos_mini

Commit message: directory clean up and better more finalized layout
Parts:
- added J6: +12V_IN, Connector_PinHeader_2.54mm:PinHeader_1x02_P2.54mm_Vertical, symbol Connector:Conn_01x02_Male
- Q1, Q2, Q3: value irfz44l -> IRLZ44N
- U1: footprint (none) -> 3a_dcdc_vreg_board:8_pin_header_mount
Connections:
- wire segments 48 -> 55
- no-connect marks 13 -> 9
Changed lines of the file:
@@
 P 6550 2150
 F 0 "Q1" H 6755 2196 50  0000 L CNN
-F 1 "irfz44l" H 6755 2105 50  0000 L CNN
+F 1 "IRLZ44N" H 6755 2105 50  0000 L CNN
 F 2 "Package_TO_SOT_THT:TO-220-3_Vertical" H 6750 2250 50  0001 C CNN
 F 3 "~" H 6550 2150 50  0001 C CNN
@@
 P 6550 3650
 F 0 "Q2" H 6755 3696 50  0000 L CNN
-F 1 "irfz44l" H 6755 3605 50  0000 L CNN
+F 1 "IRLZ44N" H 6755 3605 50  0000 L CNN
 F 2 "Package_TO_SOT_THT:TO-220-3_Vertical" H 6750 3750 50  0001 C CNN
 F 3 "~" H 6550 3650 50  0001 C CNN
@@
 P 6550 5250
 F 0 "Q3" H 6755 5296 50  0000 L CNN
-F 1 "irfz44l" H 6755 5205 50  0000 L CNN
+F 1 "IRLZ44N" H 6755 5205 50  0000 L CNN
 F 2 "Package_TO_SOT_THT:TO-220-3_Vertical" H 6750 5350 50  0001 C CNN
 F 3 "~" H 6550 5250 50  0001 C CNN
@@
 L Connector:Conn_01x02_Male J2
 U 1 1 5B999B0D
-P 3800 2300
-F 0 "J2" H 3906 2478 50  0000 C CNN
-F 1 "PWR_EN" H 3906 2387 50  0000 C CNN
-F 2 "Connector_PinHeader_2.54mm:PinHeader_1x02_P2.54mm_Vertical" H 3800 2300 50  0001 C CNN
-F 3 "~" H 3800 2300 50  0001 C CNN
-	1    3800 2300
-	1    0    0    -1
-$EndComp
-Wire Wire Line
-	4000 2400 4000 2700
+P 3400 2600
+F 0 "J2" H 3506 2778 50  0000 C CNN
+F 1 "PWR_EN" H 3506 2687 50  0000 C CNN
+F 2 "Connector_PinHeader_2.54mm:PinHeader_1x02_P2.54mm_Vertical" H 3400 2600 50  0001 C CNN
+F 3 "~" H 3400 2600 50  0001 C CNN
+	1    3400 2600
+	1    0    0    -1
+$EndComp
+Wire Wire Line
+	3600 2700 4000 2700
 Connection ~ 4000 2700
 $Comp
@@
 P 7100 1750
 F 0 "J3" V 7160 1790 50  0000 L CNN
-F 1 "BUZZ_CON" V 7251 1790 50  0000 L CNN
+F 1 "BUZZ_CON" V 7050 1550 50  0000 L CNN
 F 2 "Connector_PinHeader_2.54mm:PinHeader_1x02_P2.54mm_Vertical" H 7100 1750 50  0001 C CNN
 F 3 "~" H 7100 1750 50  0001 C CNN
@@
 P 7100 3250
 F 0 "J4" H 7160 3290 50  0000 L CNN
-F 1 "VIBE_CON" V 7251 3290 50  0000 L CNN
+F 1 "VIBE_CON" V 7050 3050 50  0000 L CNN
 F 2 "Connector_PinHeader_2.54mm:PinHeader_1x02_P2.54mm_Vertical" H 7100 3250 50  0001 C CNN
 F 3 "~" H 7100 3250 50  0001 C CNN
@@
 P 7100 4850
 F 0 "J5" H 7160 4890 50  0000 L CNN
-F 1 "LED_CON" V 7200 4800 50  0000 L CNN
+F 1 "LED_CON" V 7050 4650 50  0000 L CNN
 F 2 "Connector_PinHeader_2.54mm:PinHeader_1x02_P2.54mm_Vertical" H 7100 4850 50  0001 C CNN
 F 3 "~" H 7100 4850 50  0001 C CNN
@@
 L power:PWR_FLAG #FLG0101
 U 1 1 5B9BE36E
-P 7600 2050
-F 0 "#FLG0101" H 7600 2125 50  0001 C CNN
-F 1 "PWR_FLAG" V 7600 2178 50  0000 L CNN
-F 2 "" H 7600 2050 50  0001 C CNN
-F 3 "~" H 7600 2050 50  0001 C CNN
-	1    7600 2050
-	0    1    1    0
+P 4150 1750
+F 0 "#FLG0101" H 4150 1825 50  0001 C CNN
+F 1 "PWR_FLAG" V 4150 1878 50  0000 L CNN
+F 2 "" H 4150 1750 50  0001 C CNN
+F 3 "~" H 4150 1750 50  0001 C CNN
+	1    4150 1750
+	1    0    0    -1
 $EndComp
 $Comp
@@
 F 0 "U1" H 4800 2065 50  0000 C CNN
 F 1 "3a_dcdc_vreg_board" H 4800 1974 50  0000 C CNN
-F 2 "" H 4750 1600 50  0001 C CNN
+F 2 "3a_dcdc_vreg_board:8_pin_header_mount" H 4750 1600 50  0001 C CNN
 F 3 "" H 4750 1600 50  0001 C CNN
 	1    4800 1600
@@
 L power:GND #PWR0101
 U 1 1 5B9A029B
-P 4800 2150
-F 0 "#PWR0101" H 4800 1900 50  0001 C CNN
-F 1 "GND" H 4850 2000 50  0000 R CNN
-F 2 "" H 4800 2150 50  0001 C CNN
-F 3 "" H 4800 2150 50  0001 C CNN
-	1    4800 2150
-	1    0    0    -1
+P 4800 1000
+F 0 "#PWR0101" H 4800 750 50  0001 C CNN
+F 1 "GND" H 4850 850 50  0000 R CNN
+F 2 "" H 4800 1000 50  0001 C CNN
+F 3 "" H 4800 1000 50  0001 C CNN
+	1    4800 1000
+	-1   0    0    1
 $EndComp
 $Comp
 L power:+12V #PWR0102
 U 1 1 5B9A1455
-P 4400 1400
-F 0 "#PWR0102" H 4400 1250 50  0001 C CNN
-F 1 "+12V" H 4400 1550 50  0000 C CNN
-F 2 "" H 4400 1400 50  0001 C CNN
-F 3 "" H 4400 1400 50  0001 C CNN
-	1    4400 1400
+P 4050 1750
+F 0 "#PWR0102" H 4050 1600 50  0001 C CNN
+F 1 "+12V" H 4050 1900 50  0000 C CNN
+F 2 "" H 4050 1750 50  0001 C CNN
+F 3 "" H 4050 1750 50  0001 C CNN
+	1    4050 1750
 	0    -1   -1   0
 $EndComp
@@
 L power:PWR_FLAG #FLG0102
 U 1 1 5B9A159D
-P 5200 2150
-F 0 "#FLG0102" H 5200 2225 50  0001 C CNN
-F 1 "PWR_FLAG" H 5200 2324 50  0000 C CNN
-F 2 "" H 5200 2150 50  0001 C CNN
-F 3 "~" H 5200 2150 50  0001 C CNN
-	1    5200 2150
-	0    1    1    0
-$EndComp
-Wire Wire Line
-	4400 1850 4400 2150
-Wire Wire Line
-	4400 2150 4800 2150
-Wire Wire Line
-	4800 2150 5200 2150
-Wire Wire Line
-	5200 2150 5200 1850
-Connection ~ 4800 2150
-Connection ~ 5200 2150
-Wire Wire Line
-	5200 1400 5200 1050
-Wire Wire Line
-	5200 1050 4100 1050
-Wire Wire Line
-	4100 1050 4100 2300
-Wire Wire Line
-	4100 2300 4000 2300
-NoConn ~ 5200 1500
-NoConn ~ 5200 1750
-NoConn ~ 4400 1750
-NoConn ~ 4400 1500
+P 5200 1000
+F 0 "#FLG0102" H 5200 1075 50  0001 C CNN
+F 1 "PWR_FLAG" H 5200 1174 50  0000 C CNN
+F 2 "" H 5200 1000 50  0001 C CNN
+F 3 "~" H 5200 1000 50  0001 C CNN
+	1    5200 1000
+	0    1    1    0
+$EndComp
+Wire Wire Line
+	4400 1750 4400 1850
+Connection ~ 4400 1750
+Wire Wire Line
+	5200 1750 5200 1850
+Wire Wire Line
+	5200 1400 5200 1500
+Wire Wire Line
+	4400 1400 4400 1500
+Wire Wire Line
+	4400 1400 4400 1000
+Wire Wire Line
+	4400 1000 4800 1000
+Wire Wire Line
+	5200 1000 5200 1400
+Connection ~ 4400 1400
+Connection ~ 5200 1400
+Connection ~ 4800 1000
+Wire Wire Line
+	4800 1000 5200 1000
+Connection ~ 5200 1000
+Connection ~ 5200 1850
+Wire Wire Line
+	4050 1750 4150 1750
+Connection ~ 4150 1750
+Wire Wire Line
+	4150 1750 4400 1750
+Wire Wire Line
+	5200 2600 3600 2600
+Wire Wire Line
+	5200 1850 5200 2600
+$Comp
+L Connector:Conn_01x02_Male J6
+U 1 1 5B9B47F6
+P 3400 2050
+F 0 "J6" H 3506 2228 50  0000 C CNN
+F 1 "+12V_IN" H 3506 2137 50  0000 C CNN
+F 2 "Connector_PinHeader_2.54mm:PinHeader_1x02_P2.54mm_Vertical" H 3400 2050 50  0001 C CNN
+F 3 "~" H 3400 2050 50  0001 C CNN
+	1    3400 2050
+	1    0    0    -1
+$EndComp
+Wire Wire Line
+	4150 1750 4150 2050
+Wire Wire Line
+	4150 2050 3600 2050
+$Comp
+L power:GND #PWR07
+U 1 1 5B9B5597
+P 3800 2150
+F 0 "#PWR07" H 3800 1900 50  0001 C CNN
+F 1 "GND" H 3850 2000 50  0000 R CNN
+F 2 "" H 3800 2150 50  0001 C CNN
+F 3 "" H 3800 2150 50  0001 C CNN
+	1    3800 2150
+	1    0    0    -1
+$EndComp
+Wire Wire Line
+	3800 2150 3600 2150
 $EndSCHEMATC

Commit message: Finalized board layout and added some pictures to the info
Parts:
- added J7: OFF_BTN, Connector_PinHeader_2.54mm:PinHeader_1x02_P2.54mm_Vertical, symbol Connector:Conn_01x02_Male
Connections:
- wire segments 55 -> 58
- no-connect marks 9 -> 8
Changed lines of the file:
@@
 L power:GND #PWR01
 U 1 1 5B97D6F2
-P 3600 3350
-F 0 "#PWR01" H 3600 3100 50  0001 C CNN
-F 1 "GND" H 3605 3177 50  0000 C CNN
-F 2 "" H 3600 3350 50  0001 C CNN
-F 3 "" H 3600 3350 50  0001 C CNN
-	1    3600 3350
+P 3150 3350
+F 0 "#PWR01" H 3150 3100 50  0001 C CNN
+F 1 "GND" H 3155 3177 50  0000 C CNN
+F 2 "" H 3150 3350 50  0001 C CNN
+F 3 "" H 3150 3350 50  0001 C CNN
+	1    3150 3350
 	0    -1   -1   0
 $EndComp
@@
 L Connector:Conn_01x04_Male J1
 U 1 1 5B97FFEF
-P 3400 3450
-F 0 "J1" V 3460 3163 50  0000 R CNN
-F 1 "OLED" V 3551 3163 50  0000 R CNN
-F 2 "Connector_PinHeader_2.54mm:PinHeader_1x04_P2.54mm_Vertical" H 3400 3450 50  0001 C CNN
-F 3 "~" H 3400 3450 50  0001 C CNN
-	1    3400 3450
+P 2950 3450
+F 0 "J1" V 3010 3163 50  0000 R CNN
+F 1 "OLED" V 3101 3163 50  0000 R CNN
+F 2 "Connector_PinHeader_2.54mm:PinHeader_1x04_P2.54mm_Vertical" H 2950 3450 50  0001 C CNN
+F 3 "~" H 2950 3450 50  0001 C CNN
+	1    2950 3450
 	1    0    0    -1
 $EndComp
@@
 Connection ~ 6350 2150
 Wire Wire Line
-	3600 3450 4000 3450
-Wire Wire Line
-	4000 3450 4000 2700
-Wire Wire Line
-	4000 2700 5800 2700
+	3150 3450 3600 3450
+Wire Wire Line
+	3600 3450 3600 2700
+Wire Wire Line
+	3600 2700 5800 2700
 Wire Wire Line
 	5800 2700 5800 3250
@@
 	5800 3250 5450 3250
 Wire Wire Line
-	3600 3550 3750 3550
-Wire Wire Line
-	3750 3550 3750 3750
-Wire Wire Line
-	3750 3750 4450 3750
-Wire Wire Line
-	4450 3650 3600 3650
+	3150 3550 3300 3550
+Wire Wire Line
+	3300 3550 3300 3750
+Wire Wire Line
+	3300 3750 4450 3750
+Wire Wire Line
+	4450 3650 3150 3650
 $Comp
 L power:GND #PWR02
 U 1 1 5B996D77
-P 4450 3350
-F 0 "#PWR02" H 4450 3100 50  0001 C CNN
-F 1 "GND" H 4455 3177 50  0000 C CNN
-F 2 "" H 4450 3350 50  0001 C CNN
-F 3 "" H 4450 3350 50  0001 C CNN
-	1    4450 3350
-	0    1    1    0
+P 4250 3350
+F 0 "#PWR02" H 4250 3100 50  0001 C CNN
+F 1 "GND" H 4255 3177 50  0000 C CNN
+F 2 "" H 4250 3350 50  0001 C CNN
+F 3 "" H 4250 3350 50  0001 C CNN
+	1    4250 3350
+	-1   0    0    1
 $EndComp
 $Comp
@@
 	1    0    0    -1
 $EndComp
-Wire Wire Line
-	3600 2700 4000 2700
-Connection ~ 4000 2700
 $Comp
 L Connector:Conn_01x02_Male J3
@@
 NoConn ~ 4450 3950
 NoConn ~ 4450 3850
-NoConn ~ 4450 3550
-NoConn ~ 4450 3450
 NoConn ~ 4450 3250
 Wire Wire Line
@@
 Wire Wire Line
 	3800 2150 3600 2150
+$Comp
+L Connector:Conn_01x02_Male J7
+U 1 1 5B9AD0E4
+P 3850 3550
+F 0 "J7" H 3750 3500 50  0000 C CNN
+F 1 "OFF_BTN" H 3950 3350 50  0000 C CNN
+F 2 "Connector_PinHeader_2.54mm:PinHeader_1x02_P2.54mm_Vertical" H 3850 3550 50  0001 C CNN
+F 3 "~" H 3850 3550 50  0001 C CNN
+	1    3850 3550
+	1    0    0    1
+$EndComp
+Connection ~ 3600 2700
+NoConn ~ 4450 3450
+Wire Wire Line
+	4050 3550 4450 3550
+Wire Wire Line
+	4050 3450 4250 3450
+Wire Wire Line
+	4250 3450 4250 3350
+Wire Wire Line
+	4450 3350 4250 3350
+Connection ~ 4250 3350
 $EndSCHEMATC
